File: LIC_rack_CV-01.sch (EAGLE design)
At the start: 53 parts, among them IC1 TS1117, IC2 MEGA32-A, IC3 MEGA8-AI, IC6 MAX481CSA, Q1 BSS138, Q2 14.7456, Q3 BSS138, Q4 14.7456, Q5 BSS138, Q6 BSS138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

Commit message: Dalsi verze
Upravena deska skrz SS pin
Connections:
- removed net N$4: IC2.(SS)PB4
- net PX_IRQ: no longer IC2.(AIN0/INT2)PB2
- net PX_IRQ_RFID: no longer J1-A18.MS
- net PX_SS: now also IC2.(SS)PB4; no longer IC2.(INT1)PD3
Other:
- note added: "Zmena-> Upraven pin z PB2 na PB4 pro ovládání SS"
Changed lines of the file:
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@@
 <sheet>
 <plain>
+<text x="162.56" y="5.08" size="1.016" layer="94">Zmena-&gt; Upraven pin z PB2 na PB4
+pro ovládání SS</text>
 </plain>
 <instances>
@@
 <net name="PX_SS" class="0">
 <segment>
-<pinref part="IC2" gate="G$1" pin="(INT1)PD3"/>
-<wire x1="91.44" y1="73.66" x2="96.52" y2="73.66" width="0.1524" layer="91"/>
-<label x="96.52" y="73.66" size="1.016" layer="95" xref="yes"/>
+<pinref part="IC2" gate="G$1" pin="(SS)PB4"/>
+<wire x1="91.44" y1="121.92" x2="96.52" y2="121.92" width="0.1524" layer="91"/>
+<label x="96.52" y="121.92" size="1.27" layer="95" font="vector" ratio="12" xref="yes"/>
 </segment>
 </net>
@@
 <wire x1="226.06" y1="93.98" x2="233.68" y2="93.98" width="0.1524" layer="91"/>
 <label x="233.68" y="93.98" size="1.016" layer="95" xref="yes"/>
-</segment>
-</net>
-<net name="PX_IRQ" class="0">
-<segment>
-<pinref part="IC2" gate="G$1" pin="(AIN0/INT2)PB2"/>
-<wire x1="91.44" y1="116.84" x2="96.52" y2="116.84" width="0.1524" layer="91"/>
-<label x="96.52" y="116.84" size="1.016" layer="95" xref="yes"/>
-</segment>
-</net>
-<net name="N$4" class="0">
-<segment>
-<pinref part="IC2" gate="G$1" pin="(SS)PB4"/>
-<wire x1="91.44" y1="121.92" x2="96.52" y2="121.92" width="0.1524" layer="91"/>
 </segment>
 </net>
@@
 </segment>
 </net>
-<net name="PX_IRQ_RFID" class="0">
-<segment>
-<pinref part="J1" gate="-A18" pin="MS"/>
-<wire x1="220.98" y1="114.3" x2="205.74" y2="114.3" width="0.1524" layer="91"/>
-<label x="205.74" y="114.3" size="1.016" layer="95" rot="R180" xref="yes"/>
-</segment>
-</net>
 <net name="RXD_RFID" class="0">
 <segment>
@@
 </schematic>
 </drawing>
+<compatibility>
+<note version="6.3" minversion="6.2.2" severity="warning">
+Since Version 6.2.2 text objects can contain more than one line,
+which will not be processed correctly with this version.
+</note>
+</compatibility>
 </eagle>
